File: hardware/vectrex-led.kicad_pcb (KiCad board)
At the start: 2 copper layers, 35.5 x 15.2 mm, 10 parts, among them SW1 SW_DIP_x03

Commit message: migrate 3D shapes to built-in KiCad 6.x location
Other:
- net class Default removed
- net class Large removed
